File: LED-Treiber/Treiber.kicad_pcb (KiCad board)
At the start: 2 copper layers, 279.5 x 36.6 mm, 46 parts, among them J1 Conn_01x01_Female, J2 Conn_01x01_Female, J3 Conn_01x01_Female, J4 Conn_01x01_Female, J5 Conn_01x01_Female, J6 Conn_01x01_Female, U1 TPS92200DxRXL

Commit message: Swapped some LED's
Parts:
- moved D17 34.8 mm to (169.2, 94.5)
- moved D5 23.2 mm to (308.5, 94.5)
- moved D8 23.2 mm to (273.7, 94.5)
- moved D15 23.2 mm to (192.4, 94.5)
- moved D19 23.2 mm to (146.0, 94.5)
- moved D23 23.2 mm to (99.6, 94.5)
- moved D22 23.2 mm to (111.2, 94.5)
- moved D10 11.6 mm to (250.5, 94.5)
- moved D9 11.6 mm to (262.1, 94.5)
- moved D14 11.6 mm to (204.1, 94.5)
- moved D20 11.6 mm to (134.4, 94.5)
- moved D3 11.6 mm to (331.8, 94.5)
- moved D4 11.6 mm to (320.1, 94.5)
- moved D6 11.6 mm to (296.9, 94.5)
- moved D7 11.6 mm to (285.3, 94.5)
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Changed lines of the file:
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@@
   (net 12 "Net-(J3-Pad1)")
   (footprint "LED_SMD:LED_PLCC_2835" (layer "F.Cu")
-    (at 320.15 94.5)
+    (at 331.76 94.5)
     (descr "https://www.luckylight.cn/media/component/data-sheet/R2835BC-B2M-M10.pdf")
     (tags "LED")
@@
   )
   (footprint "LED_SMD:LED_PLCC_2835" (layer "F.Cu")
-    (at 250.49 94.5)
+    (at 262.11 94.5)
     (descr "https://www.luckylight.cn/media/component/data-sheet/R2835BC-B2M-M10.pdf")
     (tags "LED")
@@
   )
   (footprint "LED_SMD:LED_PLCC_2835" (layer "F.Cu")
-    (at 134.39 94.5)
+    (at 169.22 94.5)
     (descr "https://www.luckylight.cn/media/component/data-sheet/R2835BC-B2M-M10.pdf")
     (tags "LED")
@@
   )
   (footprint "LED_SMD:LED_PLCC_2835" (layer "F.Cu")
-    (at 331.76 94.5)
+    (at 320.15 94.5)
     (descr "https://www.luckylight.cn/media/component/data-sheet/R2835BC-B2M-M10.pdf")
     (tags "LED")
@@
   )
   (footprint "LED_SMD:LED_PLCC_2835" (layer "F.Cu")
-    (at 262.11 94.5)
+    (at 250.49 94.5)
     (descr "https://www.luckylight.cn/media/component/data-sheet/R2835BC-B2M-M10.pdf")
     (tags "LED")
@@
   )
   (footprint "LED_SMD:LED_PLCC_2835" (layer "F.Cu")
-    (at 88 94.5)
+    (at 111.17 94.5)
     (descr "https://www.luckylight.cn/media/component/data-sheet/R2835BC-B2M-M10.pdf")
     (tags "LED")
@@
   )
   (footprint "LED_SMD:LED_PLCC_2835" (layer "F.Cu")
-    (at 285.32 94.5)
+    (at 308.54 94.5)
     (descr "https://www.luckylight.cn/media/component/data-sheet/R2835BC-B2M-M10.pdf")
     (tags "LED")
@@
   )
   (footprint "LED_SMD:LED_PLCC_2835" (layer "F.Cu")
-    (at 99.56 94.5)
+    (at 88 94.5)
     (descr "https://www.luckylight.cn/media/component/data-sheet/R2835BC-B2M-M10.pdf")
     (tags "LED")
@@
   )
   (footprint "LED_SMD:LED_PLCC_2835" (layer "F.Cu")
-    (at 215.66 94.5)
+    (at 192.44 94.5)
     (descr "https://www.luckylight.cn/media/component/data-sheet/R2835BC-B2M-M10.pdf")
     (tags "LED")
@@
   )
   (footprint "LED_SMD:LED_PLCC_2835" (layer "F.Cu")
-    (at 169.22 94.5)
+    (at 146 94.5)
     (descr "https://www.luckylight.cn/media/component/data-sheet/R2835BC-B2M-M10.pdf")
     (tags "LED")
@@
   )
   (footprint "LED_SMD:LED_PLCC_2835" (layer "F.Cu")
-    (at 122.78 94.5)
+    (at 99.56 94.5)
     (descr "https://www.luckylight.cn/media/component/data-sheet/R2835BC-B2M-M10.pdf")
     (tags "LED")
@@
   )
   (footprint "LED_SMD:LED_PLCC_2835" (layer "F.Cu")
-    (at 192.44 94.5)
+    (at 204.05 94.5)
     (descr "https://www.luckylight.cn/media/component/data-sheet/R2835BC-B2M-M10.pdf")
     (tags "LED")
@@
   )
   (footprint "LED_SMD:LED_PLCC_2835" (layer "F.Cu")
-    (at 146 94.5)
+    (at 134.39 94.5)
     (descr "https://www.luckylight.cn/media/component/data-sheet/R2835BC-B2M-M10.pdf")
     (tags "LED")
@@
   )
   (footprint "LED_SMD:LED_PLCC_2835" (layer "F.Cu")
-    (at 204.05 94.5)
+    (at 215.66 94.5)
     (descr "https://www.luckylight.cn/media/component/data-sheet/R2835BC-B2M-M10.pdf")
     (tags "LED")
@@
   )
   (footprint "LED_SMD:LED_PLCC_2835" (layer "F.Cu")
-    (at 308.54 94.5)
+    (at 296.93 94.5)
     (descr "https://www.luckylight.cn/media/component/data-sheet/R2835BC-B2M-M10.pdf")
     (tags "LED")
@@
   )
   (footprint "LED_SMD:LED_PLCC_2835" (layer "F.Cu")
-    (at 273.71 94.5)
+    (at 285.32 94.5)
     (descr "https://www.luckylight.cn/media/component/data-sheet/R2835BC-B2M-M10.pdf")
     (tags "LED")
@@
   )
   (footprint "LED_SMD:LED_PLCC_2835" (layer "F.Cu")
-    (at 296.93 94.5)
+    (at 273.71 94.5)
     (descr "https://www.luckylight.cn/media/component/data-sheet/R2835BC-B2M-M10.pdf")
     (tags "LED")
@@
   )
   (footprint "LED_SMD:LED_PLCC_2835" (layer "F.Cu")
-    (at 111.17 94.5)
+    (at 122.78 94.5)
     (descr "https://www.luckylight.cn/media/component/data-sheet/R2835BC-B2M-M10.pdf")
     (tags "LED")
@@
   (segment (start 102.1 106.7) (end 95.9 106.7) (width 0.2) (layer "F.Cu") (net 5))
   (segment (start 114 106.7) (end 125.2 106.7) (width 0.2) (layer "F.Cu") (net 5))
-  (segment (start 156.3 106.5) (end 156.1 106.3) (width 1) (layer "F.Cu") (net 5))
   (segment (start 227 106.3) (end 302.4 106.3) (width 1.6) (layer "F.Cu") (net 5))
   (segment (start 112.545 94.5) (end 112.545 105.245) (width 0.2) (layer "F.Cu") (net 5))
@@
   (segment (start 114 106.7) (end 102.1 106.7) (width 0.2) (layer "F.Cu") (net 5))
   (segment (start 139.1 106.3) (end 136.6 103.8) (width 1.6) (layer "F.Cu") (net 5))
+  (segment (start 161.1 106.6) (end 156.4 106.6) (width 1) (layer "F.Cu") (net 5))
   (segment (start 315.1 106.2) (end 334.6 106.2) (width 1.6) (layer "F.Cu") (net 5))
+  (segment (start 156.4 106.6) (end 156.1 106.3) (width 1) (layer "F.Cu") (net 5))
   (segment (start 312.7 103.8) (end 315.1 106.2) (width 1.6) (layer "F.Cu") (net 5))
   (segment (start 224.5 103.8) (end 227 106.3) (width 1.6) (layer "F.Cu") (net 5))
@@
   (segment (start 124.155 106.7) (end 124.155 94.5) (width 0.2) (layer "F.Cu") (net 5))
   (segment (start 302.4 106.3) (end 304.9 103.8) (width 1.6) (layer "F.Cu") (net 5))
+  (segment (start 161.4 106.3) (end 161.1 106.6) (width 1) (layer "F.Cu") (net 5))
   (segment (start 348.775 103.425) (end 339.783 103.425) (width 0.2) (layer "F.Cu") (net 5))
-  (segment (start 161.4 106.3) (end 161.2 106.5) (width 1) (layer "F.Cu") (net 5))
   (segment (start 304.9 103.8) (end 312.7 103.8) (width 1.6) (layer "F.Cu") (net 5))
   (segment (start 348.8 103.4) (end 348.775 103.425) (width 0.2) (layer "F.Cu") (net 5))
@@
   (segment (start 161.4 106.3) (end 214.4 106.3) (width 1.6) (layer "F.Cu") (net 5))
   (segment (start 128.1 103.8) (end 128 103.7) (width 1.6) (layer "F.Cu") (net 5))
-  (segment (start 161.2 106.5) (end 156.3 106.5) (width 1) (layer "F.Cu") (net 5))
   (segment (start 100.935 105.535) (end 102.1 106.7) (width 0.2) (layer "F.Cu") (net 5))
   (segment (start 333.2 106.7) (end 336.475 103.425) (width 0.2) (layer "F.Cu") (net 5))
@@
         (xy 314.2 93.4)
         (xy 314.2 104)
-        (xy 313 102.8)
+        (xy 313 102.9)
         (xy 304.4 102.9)
         (xy 302 105.3)
@@
     (polygon
       (pts
-        (xy 157.8 105.9)
-        (xy 160.1 105.9)
-        (xy 160.5 105.5)
+        (xy 158.8 105.9)
+        (xy 159.3 105.9)
+        (xy 160.3 105.5)
         (xy 161.5 105.5)
         (xy 161.5 107.1)
         (xy 156 107.1)
         (xy 156 105.5)
-        (xy 157.4 105.5)
+        (xy 157.6 105.5)
       )
     )

Commit message: wip
Parts:
- L1: value 22µ -> 15µ; footprint Inductor_SMD:L_Taiyo-Yuden_NR-60xx -> Inductor_SMD:L_Taiyo-Yuden_NR-50xx
- moved L1 0.77 mm to (340.3, 105.2)
Routing:
- net Net-(C3-Pad2): track 6.50 -> 4.91 mm
Other:
- board text added: "+"
- board text added: "-"
- board text added: "P"
- board text removed: "24V"
- board text removed: "GND"
- board text removed: "PWM"
Changed lines of the file:
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@@
   (net 10 "Net-(D13-Pad2)")
   (net 11 "Net-(D17-Pad2)")
-  (net 12 "Net-(J3-Pad1)")
+  (net 12 "Net-(D25-Pad1)")
   (footprint "LED_SMD:LED_PLCC_2835" (layer "F.Cu")
     (at 331.76 94.5)
@@
     )
   )
-  (footprint "Inductor_SMD:L_Taiyo-Yuden_NR-60xx" (layer "F.Cu")
-    (at 339.783 105.775 90)
-    (descr "Inductor, Taiyo Yuden, NR series, Taiyo-Yuden_NR-60xx, 6.0mmx6.0mm")
+  (footprint "Inductor_SMD:L_Taiyo-Yuden_NR-50xx" (layer "F.Cu")
+    (at 340.3 105.2 90)
+    (descr "Inductor, Taiyo Yuden, NR series, Taiyo-Yuden_NR-50xx, 4.9mmx4.9mm")
     (tags "inductor taiyo-yuden nr smd")
-    (property "HTN" "NR6045T220M")
-    (property "Sheetfile" "Treiber.kicad_sch")
-    (property "Sheetname" "")
-    (attr smd)
-    (fp_text reference "L1" (at -0.025 -0.183 90) (layer "F.SilkS")
-      (effects (font (size 1 1) (thickness 0.15)))
-    )
-    (fp_text value "22µ" (at 0 4.5 90) (layer "F.Fab")
+    (property "HTN" "NRS5030T150M")
+    (property "Sheetfile" "Treiber.kicad_sch")
+    (property "Sheetname" "")
+    (attr smd)
+    (fp_text reference "L1" (at 0 -3.45 90) (layer "F.SilkS")
+      (effects (font (size 1 1) (thickness 0.15)))
+    )
+    (fp_text value "15µ" (at 0 3.95 90) (layer "F.Fab")
       (effects (font (size 1 1) (thickness 0.15)))
     )
@@
       (effects (font (size 1 1) (thickness 0.15)))
     )
-    (fp_line (start -3.15 -3.1) (end 3.15 -3.1) (layer "F.SilkS") (width 0.12))
-    (fp_line (start -3.15 3.1) (end 3.15 3.1) (layer "F.SilkS") (width 0.12))
-    (fp_line (start -3.45 -3.25) (end -3.45 3.25) (layer "F.CrtYd") (width 0.05))
-    (fp_line (start 3.45 3.25) (end 3.45 -3.25) (layer "F.CrtYd") (width 0.05))
-    (fp_line (start -3.45 3.25) (end 3.45 3.25) (layer "F.CrtYd") (width 0.05))
-    (fp_line (start 3.45 -3.25) (end -3.45 -3.25) (layer "F.CrtYd") (width 0.05))
-    (fp_line (start -3 2) (end -2 3) (layer "F.Fab") (width 0.1))
-    (fp_line (start -3 2) (end -3 -2) (layer "F.Fab") (width 0.1))
-    (fp_line (start 3 2) (end 3 -2) (layer "F.Fab") (width 0.1))
-    (fp_line (start -2 3) (end 2 3) (layer "F.Fab") (width 0.1))
-    (fp_line (start -3 -2) (end -2 -3) (layer "F.Fab") (width 0.1))
-    (fp_line (start 3 -2) (end 2 -3) (layer "F.Fab") (width 0.1))
-    (fp_line (start -2 -3) (end 2 -3) (layer "F.Fab") (width 0.1))
-    (fp_line (start 3 2) (end 2 3) (layer "F.Fab") (width 0.1))
-    (pad "1" smd rect (at -2.35 0 90) (size 1.6 5.7) (layers "F.Cu" "F.Paste" "F.Mask")
+    (fp_line (start -2.55 2.55) (end 2.55 2.55) (layer "F.SilkS") (width 0.12))
+    (fp_line (start -2.55 -2.55) (end 2.55 -2.55) (layer "F.SilkS") (width 0.12))
+    (fp_line (start 2.8 -2.75) (end -2.8 -2.75) (layer "F.CrtYd") (width 0.05))
+    (fp_line (start -2.8 2.75) (end 2.8 2.75) (layer "F.CrtYd") (width 0.05))
+    (fp_line (start -2.8 -2.75) (end -2.8 2.75) (layer "F.CrtYd") (width 0.05))
+    (fp_line (start 2.8 2.75) (end 2.8 -2.75) (layer "F.CrtYd") (width 0.05))
+    (fp_line (start -1.65 -2.45) (end 1.65 -2.45) (layer "F.Fab") (width 0.1))
+    (fp_line (start 2.45 1.65) (end 1.65 2.45) (layer "F.Fab") (width 0.1))
+    (fp_line (start -1.65 2.45) (end 1.65 2.45) (layer "F.Fab") (width 0.1))
+    (fp_line (start -2.45 1.65) (end -1.65 2.45) (layer "F.Fab") (width 0.1))
+    (fp_line (start 2.45 -1.65) (end 1.65 -2.45) (layer "F.Fab") (width 0.1))
+    (fp_line (start -2.45 -1.65) (end -1.65 -2.45) (layer "F.Fab") (width 0.1))
+    (fp_line (start 2.45 -1.65) (end 2.45 1.65) (layer "F.Fab") (width 0.1))
+    (fp_line (start -2.45 1.65) (end -2.45 -1.65) (layer "F.Fab") (width 0.1))
+    (pad "1" smd rect (at -1.8 0 90) (size 1.5 4) (layers "F.Cu" "F.Paste" "F.Mask")
       (net 4 "Net-(C3-Pad2)") (pinfunction "1") (pintype "passive"))
-    (pad "2" smd rect (at 2.35 0 90) (size 1.6 5.7) (layers "F.Cu" "F.Paste" "F.Mask")
+    (pad "2" smd rect (at 1.8 0 90) (size 1.5 4) (layers "F.Cu" "F.Paste" "F.Mask")
       (net 5 "Net-(C4-Pad2)") (pinfunction "2") (pintype "passive"))
-    (model "${KICAD6_3DMODEL_DIR}/Inductor_SMD.3dshapes/L_Taiyo-Yuden_NR-60xx.wrl"
+    (model "${KICAD6_3DMODEL_DIR}/Inductor_SMD.3dshapes/L_Taiyo-Yuden_NR-50xx.wrl"
       (offset (xyz 0 0 0))
       (scale (xyz 1 1 1))
@@
     (fp_line (start -0.3 0) (end 0.2 -0.35) (layer "F.Fab") (width 0.1))
     (pad "1" smd rect (at -1.05 0 270) (size 0.6 0.45) (layers "F.Cu" "F.Paste" "F.Mask")
-      (net 12 "Net-(J3-Pad1)") (pinfunction "K") (pintype "passive"))
+      (net 12 "Net-(D25-Pad1)") (pinfunction "K") (pintype "passive"))
     (pad "2" smd rect (at 1.05 0 270) (size 0.6 0.45) (layers "F.Cu" "F.Paste" "F.Mask")
       (net 1 "GND") (pinfunction "A") (pintype "passive"))
@@
     )
     (pad "1" smd roundrect (at 0 0) (size 2 1) (layers "F.Cu" "F.Mask") (roundrect_rratio 0.25)
-      (net 12 "Net-(J3-Pad1)") (pinfunction "Pin_1") (pintype "passive"))
+      (net 12 "Net-(D25-Pad1)") (pinfunction "Pin_1") (pintype "passive"))
   )
   (footprint "Bergi:VQFN-HR" (layer "F.Cu")
@@
       (net 1 "GND") (pinfunction "GND") (pintype "unspecified") (solder_mask_margin 0.05))
     (pad "5" smd roundrect (at 0.65 -0.275) (size 0.6 0.2) (layers "F.Cu" "F.Paste" "F.Mask") (roundrect_rratio 0.25)
-      (net 12 "Net-(J3-Pad1)") (pinfunction "DIM") (pintype "unspecified") (solder_mask_margin 0.05))
+      (net 12 "Net-(D25-Pad1)") (pinfunction "DIM") (pintype "unspecified") (solder_mask_margin 0.05))
     (pad "6" smd custom (at 0.45 -0.775) (size 0 0) (layers "F.Cu" "F.Mask")
       (net 6 "Net-(D1-Pad1)") (pinfunction "FB") (pintype "unspecified") (solder_mask_margin 0.05)
@@
       (net 2 "Net-(C1-Pad2)") (pintype "passive"))
     (pad "2" smd roundrect (at 0.825 0 90) (size 0.8 0.95) (layers "F.Cu" "F.Paste" "F.Mask") (roundrect_rratio 0.25)
-      (net 12 "Net-(J3-Pad1)") (pintype "passive"))
+      (net 12 "Net-(D25-Pad1)") (pintype "passive"))
     (model "${KICAD6_3DMODEL_DIR}/Resistor_SMD.3dshapes/R_0603_1608Metric.wrl"
       (offset (xyz 0 0 0))
@@
     )
     (pad "1" smd roundrect (at 0 0) (size 2 1) (layers "F.Cu" "F.Mask") (roundrect_rratio 0.25)
-      (net 12 "Net-(J3-Pad1)") (pinfunction "Pin_1") (pintype "passive"))
+      (net 12 "Net-(D25-Pad1)") (pinfunction "Pin_1") (pintype "passive"))
   )
   (footprint "Resistor_SMD:R_0603_1608Metric" (layer "F.Cu")
@@
   (gr_line (start 83.5 76.2) (end 83.5 79) (layer "Edge.Cuts") (width 0.1))
   (gr_line (start 83.5 79) (end 82 79) (layer "Edge.Cuts") (width 0.1))
-  (gr_text "GND" (at 356.8 80.5) (layer "F.SilkS")
-    (effects (font (size 1 1) (thickness 0.15)))
-  )
-  (gr_text "PWM" (at 88.1 105.5) (layer "F.SilkS")
-    (effects (font (size 1.5 1.5) (thickness 0.3)))
-  )
-  (gr_text "PWM" (at 358.4 103.1) (layer "F.SilkS")
-    (effects (font (size 1.5 1.5) (thickness 0.3)))
-  )
-  (gr_text "GND" (at 87.6 80.6) (layer "F.SilkS")
-    (effects (font (size 1.5 1.5) (thickness 0.3)))
-  )
-  (gr_text "24V" (at 87.8 108.5) (layer "F.SilkS")
-    (effects (font (size 1.5 1.5) (thickness 0.3)))
-  )
-  (gr_text "24V" (at 356.3 108.5) (layer "F.SilkS")
-    (effects (font (size 1.5 1.5) (thickness 0.3)))
+  (gr_text "-" (at 357.2 80.3) (layer "F.SilkS")
+    (effects (font (size 2 2) (thickness 0.3)))
+  )
+  (gr_text "P" (at 87 105.6) (layer "F.SilkS")
+    (effects (font (size 2 2) (thickness 0.3)))
+  )
+  (gr_text "P" (at 357.4 105.4) (layer "F.SilkS")
+    (effects (font (size 2 2) (thickness 0.3)))
+  )
+  (gr_text "-" (at 87.2 80.3) (layer "F.SilkS")
+    (effects (font (size 2 2) (thickness 0.3)))
+  )
+  (gr_text "+" (at 86.9 108.4) (layer "F.SilkS")
+    (effects (font (size 2 2) (thickness 0.3)))
+  )
+  (gr_text "+" (at 356.9 108.2) (layer "F.SilkS")
+    (effects (font (size 2 2) (thickness 0.3)))
   )
   (dimension (type aligned) (layer "Dwgs.User")
@@
   (segment (start 344.283 104.937) (end 343.7 104.354) (width 0.2) (layer "F.Cu") (net 3))
   (segment (start 345.279 104.937) (end 344.283 104.937) (width 0.2) (layer "F.Cu") (net 3))
-  (segment (start 341.479 108.125) (end 339.783 108.125) (width 0.2) (layer "F.Cu") (net 4))
-  (segment (start 343.7 105.904) (end 341.479 108.125) (width 0.2) (layer "F.Cu") (net 4))
+  (segment (start 344.017 105.587) (end 342.604 107) (width 0.2) (layer "F.Cu") (net 4))
   (segment (start 345.229 105.587) (end 344.017 105.587) (width 0.2) (layer "F.Cu") (net 4))
-  (segment (start 344.017 105.587) (end 343.7 105.904) (width 0.2) (layer "F.Cu") (net 4))
+  (segment (start 342.604 107) (end 340.908 107) (width 0.2) (layer "F.Cu") (net 4))
   (segment (start 136.6 103.8) (end 128.1 103.8) (width 1.6) (layer "F.Cu") (net 5))
   (segment (start 216.9 103.8) (end 224.5 103.8) (width 1.6) (layer "F.Cu") (net 5))
@@
         (xy 312.2 104.8)
         (xy 314.7 107.3)
-        (xy 334.7 107.3)
-        (xy 336.6 109.2)
-        (xy 343.3 109.2)
+        (xy 337.2 107.3)
+        (xy 338.8 108.9)
+        (xy 343.6 108.9)
         (xy 344.4 108.1)
         (xy 344.4 106.7)
@@
         (xy 344.1 107.9)
         (xy 343.4 108.6)
-        (xy 342.6 108.6)
-        (xy 337 107.7)
-        (xy 337 106.5)
-        (xy 341.9 106.5)
+        (xy 339.3 108.6)
+        (xy 338.4 107.7)
+        (xy 338.4 106.3)
+        (xy 342.1 106.3)
         (xy 343.1 105.3)
         (xy 345.5 105.3)
