File: LED-Treiber/Treiber.kicad_sch (KiCad schematic)
At the start: 46 parts, among them J1 Conn_01x01_Female, J2 Conn_01x01_Female, J3 Conn_01x01_Female, J4 Conn_01x01_Female, J5 Conn_01x01_Female, J6 Conn_01x01_Female, U1 TPS92200DxRXL

Commit message: wip
Parts:
- L1: value 22µ -> 15µ; footprint Inductor_SMD:L_Taiyo-Yuden_NR-60xx -> Inductor_SMD:L_Taiyo-Yuden_NR-50xx; HTN NR6045T220M -> NRS5030T150M
Connections:
- net +24V: now reaches C1.2, C2.2, J1.1 (Pin_1), J2.1 (Pin_1), R2.1, U1.3 (VIN)
Other:
- moved on the sheet: C1, C2, C3, C4, D1, D10, D11, D12, D13, D14, D15, D16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
