File: LED-Steuerung/Steuerung.kicad_pcb (KiCad board)
At the start: 4 copper layers, 45 x 36.6 mm, 47 parts, among them J1 DNP, J10 Barrel_Jack_Switch, J2 Conn_02x03_Odd_Even, J3 DNP, J4 Conn_01x01_Female, J7 Conn_01x01_Female, J8 Conn_01x01_Female, SW1 SW_Push, U1 STM32WB5MMG, U2 L7983, U3 INA186A3IDDF, U4 74AHCT1G125

Commit message: removed unneeded via
Parts:
- R11: moved to B.Cu
- moved R11 0.81 mm to (181.7, 81.7)
Routing:
- net GND: track 51.6 -> 52.4 mm, vias 266 -> 265
- net Net-(R11-Pad2): track 0.57 -> 1.22 mm, vias 0 -> 1
